File: kicad/electric.kicad_sch (KiCad schematic)
At the start: 13 parts, among them U1 NodeMCU1.0(ESP-12E), U2 LM7805_TO220

Commit message: fix(kicad): added pullup on pwm control because of be quiet
Signed-off-by: Mario-F <github@fritschen.net>
Parts:
- added R4: 10k, symbol Device:R
- R3: value (none) -> 10k
Connections:
- net +5V: now also R4.1
- net at JFan.4 (Pin_4), Q?.1 (C): now also R4.2
Changed lines of the file:
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@@
   (junction (at 127 22.86) (diameter 0) (color 0 0 0 0)
   )
+  (junction (at 97.79 66.04) (diameter 0) (color 0 0 0 0)
+  )
   (junction (at 44.45 25.4) (diameter 0) (color 0 0 0 0)
   )
@@
     (stroke (width 0) (type default) (color 0 0 0 0))
   )
+  (wire (pts (xy 109.22 66.04) (xy 111.76 66.04))
+    (stroke (width 0) (type default) (color 0 0 0 0))
+  )
   (wire (pts (xy 124.46 27.94) (xy 132.08 27.94))
     (stroke (width 0) (type default) (color 0 0 0 0))
@@
     (stroke (width 0) (type default) (color 0 0 0 0))
   )
-  (wire (pts (xy 97.79 34.29) (xy 97.79 80.01))
+  (wire (pts (xy 97.79 34.29) (xy 97.79 66.04))
     (stroke (width 0) (type default) (color 0 0 0 0))
   )
@@
     (stroke (width 0) (type default) (color 0 0 0 0))
   )
+  (wire (pts (xy 97.79 66.04) (xy 97.79 80.01))
+    (stroke (width 0) (type default) (color 0 0 0 0))
+  )
   (wire (pts (xy 67.31 21.59) (xy 67.31 24.13))
     (stroke (width 0) (type default) (color 0 0 0 0))
@@
   )
   (wire (pts (xy 92.71 88.9) (xy 95.25 88.9))
+    (stroke (width 0) (type default) (color 0 0 0 0))
+  )
+  (wire (pts (xy 97.79 66.04) (xy 101.6 66.04))
     (stroke (width 0) (type default) (color 0 0 0 0))
   )
@@
     (pin "1")
   )
+  (symbol (lib_id "power:+5V") (at 111.76 66.04 270) (unit 1)
+    (in_bom yes) (on_board yes) (fields_autoplaced)
+    (property "Reference" "#PWR?" (id 0) (at 107.95 66.04 0)
+      (effects (font (size 1.27 1.27)) hide)
+    )
+    (property "Value" "+5V" (id 1) (at 115.57 66.0399 90)
+      (effects (font (size 1.27 1.27)) (justify left))
+    )
+    (property "Footprint" "" (id 2) (at 111.76 66.04 0)
+      (effects (font (size 1.27 1.27)) hide)
+    )
+    (property "Datasheet" "" (id 3) (at 111.76 66.04 0)
+      (effects (font (size 1.27 1.27)) hide)
+    )
+    (pin "1")
+  )
   (symbol (lib_id "power:+12V") (at 82.55 38.1 90) (unit 1)
     (in_bom yes) (on_board yes)
@@
     (pin "1")
   )
+  (symbol (lib_id "Device:R") (at 105.41 66.04 270) (unit 1)
+    (in_bom yes) (on_board yes)
+    (property "Reference" "R4" (id 0) (at 106.68 60.96 0)
+      (effects (font (size 1.27 1.27)) (justify left))
+    )
+    (property "Value" "10k" (id 1) (at 104.14 60.96 0)
+      (effects (font (size 1.27 1.27)) (justify left))
+    )
+    (property "Footprint" "" (id 2) (at 105.41 64.262 90)
+      (effects (font (size 1.27 1.27)) hide)
+    )
+    (property "Datasheet" "~" (id 3) (at 105.41 66.04 0)
+      (effects (font (size 1.27 1.27)) hide)
+    )
+    (pin "1")
+    (pin "2")
+  )
   (symbol (lib_id "Device:R") (at 88.9 88.9 270) (unit 1)
     (in_bom yes) (on_board yes)
@@
       (effects (font (size 1.27 1.27)) (justify left))
     )
-    (property "Value" "" (id 1) (at 87.63 83.82 0)
+    (property "Value" "10k" (id 1) (at 87.63 83.82 0)
       (effects (font (size 1.27 1.27)) (justify left))
     )
@@
       (reference "#PWR?") (unit 1) (value "+5V") (footprint "")
     )
+    (path "/51df22b6-e057-4f99-b98b-50c5e8bcccf5"
+      (reference "#PWR?") (unit 1) (value "+5V") (footprint "")
+    )
     (path "/6a2f84fe-599a-47a5-8319-b6961e4270c3"
       (reference "#PWR?") (unit 1) (value "+12V") (footprint "")
@@
       (reference "R3") (unit 1) (value "10k") (footprint "")
     )
+    (path "/d76ec66c-d0c1-4040-8259-8685c076073a"
+      (reference "R4") (unit 1) (value "10k") (footprint "")
+    )
     (path "/4244f2cf-53fb-48c6-88ac-de581a83aeb5"
